File: LEDWallSign.kicad_pcb (KiCad board)
At the start: 2 copper layers, 207 parts, among them J1 ISP Header, P1 Conn_WallPlug, SW1 KSR251GLFS, U1 ATmega328-AU, U100 TLC6C598-Q1, U2 RAC10-05SK, U200 TLC6C598-Q1, U300 TLC6C598-Q1, U400 TLC6C598-Q1, U500 TLC6C598-Q1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

Commit message: Fully organized parts into their subsystem categories. Also added new backup file for layout.
Parts:
- moved R749 230.5 mm to (42.9, 127.9)
- moved R750 221.6 mm to (50.5, 128.0)
- moved R640 218.2 mm to (50.6, 112.6)
- moved D641 211.0 mm to (56.1, 112.1)
- moved D750 210.1 mm to (50.0, 125.6)
- moved R641 206.1 mm to (56.5, 110.1)
- moved D752 201.0 mm to (67.2, 128.7)
- moved D857 201.0 mm to (52.8, 143.5)
- moved R752 197.8 mm to (67.7, 126.0)
- moved D642 194.5 mm to (61.4, 111.8)
- moved D749 192.3 mm to (43.1, 125.6)
- moved D856 192.2 mm to (47.2, 143.5)
- moved R644 191.7 mm to (72.3, 112.5)
- moved R754 190.4 mm to (83.7, 129.2)
- moved D645 190.3 mm to (78.4, 113.5)
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
Commit message: did some stuff, a lil routing
Parts:
- moved D748 42.6 mm to (81.3, 121.2)
- moved R748 42.6 mm to (81.4, 123.4)
- moved C391 37.2 mm to (146.0, 61.8)
- moved C691 37.2 mm to (147.5, 108.8)
- moved C890 37.2 mm to (145.2, 139.7)
- moved D103 37.2 mm to (105.3, 33.5)
- moved D211 37.2 mm to (104.6, 47.2)
- moved D213 37.2 mm to (115.0, 47.1)
- moved D319 37.2 mm to (104.6, 60.8)
- moved D537 37.2 mm to (115.7, 91.7)
- moved D753 37.2 mm to (112.7, 122.3)
- moved R106 37.2 mm to (122.0, 33.2)
- moved R191 37.2 mm to (133.2, 31.3)
- moved R193 37.2 mm to (134.7, 31.3)
- moved R211 37.2 mm to (106.5, 47.2)
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Routing:
- net /dataPin: track 0.00 -> 285.4 mm
- net /clockPin: track 0.00 -> 284.3 mm, vias 0 -> 16
- net /latch3: track 0.00 -> 164.5 mm, vias 0 -> 4
- net /latch1: track 0.00 -> 162.4 mm, vias 0 -> 6
- net /latch2: track 0.00 -> 147.5 mm, vias 0 -> 6
- net /latch4: track 0.00 -> 145.2 mm, vias 0 -> 4
- net /latch5: track 0.00 -> 123.4 mm, vias 0 -> 4
- net /latch6: track 0.00 -> 101.2 mm, vias 0 -> 4
- net /latch7: track 0.00 -> 80.6 mm, vias 0 -> 6
- net /latch8: track 0.00 -> 59.3 mm, vias 0 -> 6
- net /~RESET: track 0.00 -> 25.9 mm, vias 0 -> 2
- net /MOSI: track 0.00 -> 9.88 mm
- net /MISO: track 0.00 -> 7.07 mm
- net /SCK: track 0.00 -> 6.46 mm, vias 0 -> 2
