File: LEDWallSign.sch (KiCad schematic (older format))
At the start: 206 parts, among them U1 ATmega328-AU

Commit message: References and footprints completed. Added back up layout (of components sorted)
Going to play around with the layout now. Eventually hope to get final one done by end of this week.
Parts:
- removed C2: 100nF, symbol Device:C
- removed C?: C_Small, symbol Device:C_Small
- removed C? (x8): 100nF, symbol Device:C_Small
- removed C? (x7): 1uF, symbol Device:C_Small
- removed C?: 100n, symbol Device:C_Small
- removed C?: 10uF, symbol Device:CP1
- removed D?: LED, symbol Device:LED
- removed D? (x63): LED, LEDs:LED_0603_HandSoldering, symbol Device:LED
- removed R1: 1k, Resistors_SMD:R_0603_HandSoldering, symbol Device:R
- removed R? (x16): 10k, symbol Device:R
- removed R?: 1k, symbol Device:R
- removed R? (x16): DNP, symbol Device:R
- removed R? (x63): R, Resistors_SMD:R_0603_HandSoldering, symbol Device:R
- removed U? (x7): TLC6C598-Q1, symbol ledWallSign:TLC6C598-Q1
- added C2, C291, C391, C4, C491, C5, C591, C691, C7, C791, C891: 100nF, Capacitor_SMD:C_0603_1608Metric_Pad1.05x0.95mm_HandSolder, symbol Device:C_Small
- added C290, C3, C390, C490, C590, C690, C790, C890: 1uF, Capacitor_SMD:C_0603_1608Metric_Pad1.05x0.95mm_HandSolder, symbol Device:C_Small
- added C9: 18pF, Capacitor_SMD:C_0603_1608Metric_Pad1.05x0.95mm_HandSolder, symbol Device:C_Small
- added D101, D102, D103, D104, D105, D106, D107, D2, D208, D209, D210, D211, D212, D213, D214, D215, D316, D317, D318, D319, D320, D321, D322, D323, D424, D425, D426, D427, D428, D429, D430, D431, D532, D533, D534, D535, D536, D537, D538, D539, D640, D641, D642, D643, D644, D645, D646, D647, D748, D749, D750, D751, D752, D753, D754, D755, D856, D857, D858, D859, D860, D861, D862, D863: LED, LED_SMD:LED_0603_1608Metric_Pad1.05x0.95mm_HandSolder, symbol Device:LED
- added R101, R102, R103, R104, R105, R106, R107, R208, R209, R210, R211, R212, R213, R214, R215, R3, R316, R317, R318, R319, R320, R321, R322, R323, R424, R425, R426, R427, R428, R429, R430, R431, R5, R532, R533, R534, R535, R536, R537, R538, R539, R640, R641, R642, R643, R644, R645, R646, R647, R748, R749, R750, R751, R752, R753, R754, R755, R856, R857, R858, R859, R860, R861, R862, R863: 1k, Resistor_SMD:R_0805_2012Metric_Pad1.15x1.40mm_HandSolder, symbol Device:R
- added R191, R192, R291, R292, R391, R392, R491, R492, R591, R592, R691, R692, R791, R792, R891, R892: DNP, Resistor_SMD:R_0603_1608Metric_Pad1.05x0.95mm_HandSolder, symbol Device:R
- added R193, R290, R293, R390, R393, R4, R490, R493, R590, R593, R690, R693, R790, R793, R890, R893: 10k, Resistor_SMD:R_0603_1608Metric_Pad1.05x0.95mm_HandSolder, symbol Device:R
- added U200, U300, U400, U500, U600, U700, U800: TLC6C598-Q1, Package_SO:TSSOP-16_4.4x5mm_P0.65mm, symbol LEDWallSign-rescue:TLC6C598-Q1-ledWallSign
- C1: footprint (none) -> Capacitor_THT:CP_Radial_D5.0mm_P2.50mm
- C190, C191, C6: renamed from C?; footprint (none) -> Capacitor_SMD:C_0603_1608Metric_Pad1.05x0.95mm_HandSolder
- C8: renamed from C?; value C_Small -> 18pF; footprint (none) -> Capacitor_SMD:C_0603_1608Metric_Pad1.05x0.95mm_HandSolder
- D1: footprint LEDs:LED_0603_HandSoldering -> LED_SMD:LED_0603_1608Metric_Pad1.05x0.95mm_HandSolder
- D100: renamed from D?; footprint LEDs:LED_0603_HandSoldering -> LED_SMD:LED_0603_1608Metric_Pad1.05x0.95mm_HandSolder
- J1: renamed from J?; footprint (none) -> Connector_PinHeader_2.54mm:PinHeader_2x03_P2.54mm_Vertical
- L1: renamed from L?; footprint (none) -> Inductor_SMD:L_0603_1608Metric_Pad1.05x0.95mm_HandSolder
- P1: renamed from P?; footprint (none) -> ledWallSign-master:Qualtek 770W-X2
- R1: renamed from R2; footprint Resistors_SMD:R_2512_HandSoldering -> Resistor_SMD:R_2512_6332Metric_Pad1.52x3.35mm_HandSolder
- R100: renamed from R?; value R -> 1k; footprint Resistors_SMD:R_0603_HandSoldering -> Resistor_SMD:R_0805_2012Metric_Pad1.15x1.40mm_HandSolder
- R190: renamed from R?; footprint (none) -> Resistor_SMD:R_0603_1608Metric_Pad1.05x0.95mm_HandSolder
- R2: renamed from R3; footprint Resistors_SMD:R_2512_HandSoldering -> Resistor_SMD:R_2512_6332Metric_Pad1.52x3.35mm_HandSolder
- SW1: renamed from SW?; value SW_SPST -> KSR251GLFS; footprint (none) -> ledWallSign-master:KSR251GLFS
- U1: symbol MCU_Microchip_ATmega:ATmega328-AU -> LEDWallSign-rescue:ATmega328-AU-MCU_Microchip_ATmega
- U100: renamed from U?; footprint (none) -> Package_SO:TSSOP-16_4.4x5mm_P0.65mm; symbol ledWallSign:TLC6C598-Q1 -> LEDWallSign-rescue:TLC6C598-Q1-ledWallSign
- U2: renamed from U?; footprint (none) -> ledWallSign-master:RAC10-05SK; symbol ledWallSign:RAC10-05SK -> LEDWallSign-rescue:RAC10-05SK-ledWallSign
- Y1: renamed from Y?; footprint (none) -> ledWallSign-master:ECS-23G
Connections:
- wire segments 642 -> 648

Commit message: did some stuff, a lil routing
Parts:
- C1: symbol Device:CP1 -> LEDWallSign-rescue:CP1-Device
- C190, C191, C2, C290, C291, C3, C390, C391, C4, C490, C491, C5, C590, C591, C6, C690, C691, C7, C790, C791, C8, C890, C891, C9: symbol Device:C_Small -> LEDWallSign-rescue:C_Small-Device
- D1, D100, D101, D102, D103, D104, D105, D106, D107, D2, D208, D209, D210, D211, D212, D213, D214, D215, D316, D317, D318, D319, D320, D321, D322, D323, D424, D425, D426, D427, D428, D429, D430, D431, D532, D533, D534, D535, D536, D537, D538, D539, D640, D641, D642, D643, D644, D645, D646, D647, D748, D749, D750, D751, D752, D753, D754, D755, D856, D857, D858, D859, D860, D861, D862, D863: symbol Device:LED -> LEDWallSign-rescue:LED-Device
- J1: symbol Connector_Generic:Conn_02x03_Odd_Even -> LEDWallSign-rescue:Conn_02x03_Odd_Even-Connector_Generic
- L1: symbol Device:Ferrite_Bead -> LEDWallSign-rescue:Ferrite_Bead-Device
- P1: symbol Connector:Conn_WallPlug -> LEDWallSign-rescue:Conn_WallPlug-Connector
- R1, R100, R101, R102, R103, R104, R105, R106, R107, R190, R191, R192, R193, R2, R208, R209, R210, R211, R212, R213, R214, R215, R290, R291, R292, R293, R3, R316, R317, R318, R319, R320, R321, R322, R323, R390, R391, R392, R393, R4, R424, R425, R426, R427, R428, R429, R430, R431, R490, R491, R492, R493, R5, R532, R533, R534, R535, R536, R537, R538, R539, R590, R591, R592, R593, R640, R641, R642, R643, R644, R645, R646, R647, R690, R691, R692, R693, R748, R749, R750, R751, R752, R753, R754, R755, R790, R791, R792, R793, R856, R857, R858, R859, R860, R861, R862, R863, R890, R891, R892, R893: symbol Device:R -> LEDWallSign-rescue:R-Device
- SW1: symbol Switch:SW_SPST -> LEDWallSign-rescue:SW_SPST-Switch
- Y1: symbol Device:Crystal -> LEDWallSign-rescue:Crystal-Device
